File: ESP32-PhotoboothHub-PCB/ProPrj_New Project_2025-09-22_16-04-54_2026-09-08.kicad_sch (KiCad schematic)
At the start: 0 parts

Commit message: Fix photobooth schematic power, DMX and component footprints
Other:
- title: (none) -> Photobooth Hub
Changed lines of the file:
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@@
 	(generator_version "10.0")
 	(paper "A4")
+	(title_block
+		(title "Photobooth Hub")
+		(date "2026-09-08")
+	)
 	(sheet
 		(at 5.08 5.08)
