File: ESP32-PhotoboothHub-PCB/2_P2.kicad_sch (KiCad schematic)
At the start: 22 parts, among them K3 BRD-SS-105L, P1 WJ142R-5.08-02P-14-00A, Q1 MMBT2222A 1P, U3 100kHz, U4 MAX3485ESA, U7 6N137S

Commit message: Fix photobooth schematic power, DMX and component footprints
Parts:
- removed ?: (no value), ProPrj_New-easyedapro:, symbol ProPrj_New-easyedapro:Drawing-Symbol_A4
- added C17: 100nF / 50V, Capacitor_SMD:C_0603_1608Metric, symbol DMXFixes:C
- added C18: 10uF / 25V, Capacitor_SMD:C_0805_2012Metric, symbol DMXFixes:C
- added R28: 10k 1%, Resistor_SMD:R_0603_1608Metric, symbol DMXFixes:R_0603
- added U11: SN74LVC1G07DBVR, Package_TO_SOT_SMD:SOT-23-5, symbol DMXFixes:SN74LVC1G07DBVR
- C10, C11, C12, C13: footprint ProPrj_New-easyedapro:C0603 -> Capacitor_SMD:C_0603_1608Metric
- D2: footprint ProPrj_New-easyedapro:DO-35_BD2.0-L4.2-P8.20-D0.5-RD -> Diode_SMD:D_SOD-123
- D3: renamed from CAMERA_RESET_LED1; value NCD0805R1 -> Camera; footprint ProPrj_New-easyedapro:LED0805-R-RD -> Photobooth:LED_0805_2012Metric_A1K2; Function (none) -> Camera relay indicator; Model (none) -> NCD0805R1; Previous Reference (none) -> CAMERA_RESET_LED1
- J6: renamed from CON_DMX1; value (none) -> DMX output; footprint ProPrj_New-easyedapro:CONN-TH_KF250NH-3.5-3P -> Photobooth:PhoenixContact_SPT_1.5_3-V-3.5_1990863; Function (none) -> DMX output; LCSC Part Name 5.08mm 每排P数:3 排数:1 -> (none); Manufacturer KANGNEX(康奈克斯电气) -> Phoenix Contact; Manufacturer Part WJ142R-5.08-03P-14-00A -> 1990863; Model (none) -> SPT 1,5/3-V-3,5; Previous Reference (none) -> CON_DMX1; Supplier LCSC -> Phoenix Contact; Supplier Part C80054 -> 1990863
- J7: renamed from P1; value WJ142R-5.08-02P-14-00A -> Camera power relay; footprint ProPrj_New-easyedapro:CONN-TH_2P-P5.08_WJ142R-5.08-2P -> Photobooth:PhoenixContact_SPT_1.5_2-V-3.5_1990850; Function (none) -> Camera power relay; LCSC Part Name 5.08mm 每排P数:2 排数:1 -> (none); Manufacturer KANGNEX(康奈克斯电气) -> Phoenix Contact; Manufacturer Part WJ142R-5.08-02P-14-00A -> 1990850; Model (none) -> SPT 1,5/2-V-3,5; Previous Reference (none) -> P1; Supplier LCSC -> Phoenix Contact; Supplier Part C35616 -> 1990850
- K3: footprint ProPrj_New-easyedapro:RELAY-TH_BRD-SS-1XXL -> Photobooth:Relay_SPDT_QLRELAY_BRD-SS-105L
- Q1: footprint ProPrj_New-easyedapro:SOT-23-3_L2.9-W1.4-P1.91-LS2.6-BR -> Package_TO_SOT_SMD:SOT-23
- R13, R14, R15, R6, R7, R8: footprint ProPrj_New-easyedapro:R0603 -> Resistor_SMD:R_0603_1608Metric
- R26: value 330Ω -> 360R 1%; footprint ProPrj_New-easyedapro:R0603 -> Resistor_SMD:R_0603_1608Metric; symbol ProPrj_New-easyedapro:FRC0603F3300TS -> DMXFixes:R_0603; LCSC Part Name 330Ω ±1% 100mW 厚膜电阻 -> (none); Manufacturer UNI-ROYAL(厚声) -> UNI-ROYAL; Manufacturer Part 0603WAF3300T5E -> 0603WAF3600T5E; Supplier Part C23138 -> C25194; Tolerance (none) -> 1%
- R9: footprint ProPrj_New-easyedapro:R0603 -> Resistor_SMD:R_0603_1608Metric; now not fitted
- U3: value 100kHz -> TMR 1-0511; footprint ProPrj_New-easyedapro:PWRM-TH_4P-L11.5-W6.0-P2.54_B1503S -> Converter_DCDC:Converter_DCDC_TRACO_TMR-1-xxxx_Single_THT; symbol ProPrj_New-easyedapro:RO-0505S -> DMXFixes:TMR_1-0511; LCSC Part Name 1W定电压输入隔离非稳压输出电源模块 -> (none); Manufacturer ReSine PS(瑞鑫) -> TRACO POWER; Manufacturer Part B0505S-1W -> TMR 1-0511; Supplier Part C20617263 -> C7362907
- U4: value MAX3485ESA -> THVD1500DR; footprint ProPrj_New-easyedapro:PDIP-8_L9.6-W6.4-P2.54-LS7.6-BL -> Package_SO:SOIC-8_3.9x4.9mm_P1.27mm; symbol ProPrj_New-easyedapro:MAX3485ECN -> DMXFixes:THVD1500DR; LCSC Part Name MAX3485ESA 3.3V供电半双工低功耗RS-485收发器 -> (none); Manufacturer TWGMC(迪嘉) -> Texas Instruments; Manufacturer Part MAX3485ESA -> THVD1500DR; Supplier LCSC -> (none); Supplier Part C5279039 -> (none)
- U7: footprint ProPrj_New-easyedapro:SMT-8_L9.7-W6.6-P2.54-LS10.3-BL -> Package_DIP:SMDIP-8_W9.53mm
Connections:
- net 3.3V: now also C17.1, R28.2, U11.5 (VCC)
- net 485/TX: now also R28.1, U11.2 (A); no longer R26.1
- net DMX-GND: now also U3.6 (-VOUT), C18.2; no longer U3.3 (-VOUT), U4.1 (RO)
- net DMX-VCC: now also U7.7 (VE), C18.1
- net GND: now also C17.2, U11.3 (GND)
- new net: R26.1, U11.4 (Y)
- no-connect marks 3 -> 5
Other:
- note added: "3.3 V open-drain buffer drives 5 V optocoupler LED. R26 = 360R 1%: 7.01-14.73 mA worst-case; 3.3 V supply >= 3.0 V. Place C17 at U11."
- note added: "Camera powered by external DIN rail converter."
- note added: "Primary +5V: 4.75-5.25 V. Keep GND isolated from DMX-GND. Place C10/C11 at U7/U4; C12/C18 at U3 output."
- note added: "Regulated 5 V / 200 mA isolated supply"
- note removed: "DMX Power Isolation"
- note removed: "Removed PSU for camera, not reliable"
- title: (none) -> Photobooth Hub - Isolated DMX and camera reset
- moved on the sheet: C10, C11, C12, C13, D2, D3, J6, J7, K3, Q1, R13, R14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

Commit message: Update photobooth schematic and PCB layout
Parts:
- removed R9: 120Ω, Resistor_SMD:R_0603_1608Metric, symbol ProPrj_New-easyedapro:FRC0603J121 TS
Changed lines of the file:
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@@
-	)
-	(symbol
-		(lib_id "ProPrj_New-easyedapro:FRC0603J121 TS")
-		(at 262.89 115.57 90)
-		(unit 1)
-		(body_style 0)
-		(exclude_from_sim no)
-		(in_bom yes)
-		(on_board yes)
-		(in_pos_files yes)
-		(dnp yes)
-		(property "Reference" "R9"
-			(at 265.43 115.57 90)
-			(show_name no)
-			(do_not_autoplace no)
-			(effects
-				(font
-					(size 1.5748 1.5748)
-				)
-				(justify right top)
-			)
-		)
-		(property "Value" "120Ω"
-			(at 265.43 118.11 90)
-			(show_name no)
-			(do_not_autoplace no)
-			(effects
-				(font
-					(size 1.5748 1.5748)
-				)
-				(justify right top)
-			)
-		)
-		(property "Footprint" "Resistor_SMD:R_0603_1608Metric"
-			(at 262.89 115.57 0)
-			(hide yes)
-			(show_name no)
-			(do_not_autoplace no)
-			(effects
-				(font
-					(size 1.27 1.27)
-				)
-			)
-		)
-		(property "Datasheet" "https://atta.szlcsc.com/upload/public/pdf/source/20200306/C422600_1E6D84923E4A46A82E41ADD87F860B5C.pdf"
-			(at 262.89 115.57 0)
-			(hide yes)
-			(show_name no)
-			(do_not_autoplace no)
-			(effects
-				(font
-					(size 1.27 1.27)
-				)
-			)
-		)
-		(property "Description" "Type:Thick Film Resistors Resistance: Tolerance:±1% Tolerance:±1% Power(Watts): Overload Voltage (Max): Temperature Coefficient:±100ppm/℃ Temperature Coefficient:±100ppm/℃ Operating Temperature Range:-55℃~+155℃ Operating Temperature Range:-55℃~+155℃"
-			(at 262.89 115.57 90)
-			(hide yes)
-			(show_name no)
-			(do_not_autoplace no)
-			(effects
-				(font
-					(size 1.5748 1.5748)
-				)
-				(justify right top)
-			)
-		)
-		(property "Manufacturer Part" "0603WAF1200T5E"
-			(at 262.89 115.57 0)
-			(hide yes)
-			(show_name no)
-			(do_not_autoplace no)
-			(effects
-				(font
-					(size 1.27 1.27)
-				)
-			)
-		)
-		(property "Manufacturer" "UNI-ROYAL(厚声)"
-			(at 262.89 115.57 0)
-			(hide yes)
-			(show_name no)
-			(do_not_autoplace no)
-			(effects
-				(font
-					(size 1.27 1.27)
-				)
-			)
-		)
-		(property "Supplier Part" "C22787"
-			(at 262.89 115.57 0)
-			(hide yes)
-			(show_name no)
-			(do_not_autoplace no)
-			(effects
-				(font
-					(size 1.27 1.27)
-				)
-			)
-		)
-		(property "Supplier" "LCSC"
-			(at 262.89 115.57 0)
-			(hide yes)
-			(show_name no)
-			(do_not_autoplace no)
-			(effects
-				(font
-					(size 1.27 1.27)
-				)
-			)
-		)
-		(property "LCSC Part Name" "120Ω ±1% 100mW 厚膜电阻"
-			(at 262.89 115.57 0)
-			(hide yes)
-			(show_name no)
-			(do_not_autoplace no)
-			(effects
-				(font
-					(size 1.27 1.27)
-				)
-			)
-		)
-		(pin "1"
-		)
-		(pin "2"
-		)
-		(instances
-			(project "ProPrj_New Project_2025-09-22_16-04-54_2026-09-08"
-				(path "/1a06e780-7284-4b2d-8d1d-452e4ee14a37/32384adc-3785-4c3c-b068-de881dc2670b"
-					(reference "R9")
-					(unit 1)
-				)
-			)
-		)
 	)
 	(symbol
