File: ESP32-PhotoboothHub-PCB/ProPrj_New Project_2025-09-22_16-04-54_2026-09-08.kicad_pcb (KiCad board)
At the start: 2 copper layers, 100 x 130 mm, 60 parts, among them J1 5 V supply, J2 Command button, J3 Front lighting, J4 Printer lighting, J5 Down lighting, J6 DMX output, J7 Camera power relay, K3 BRD-SS-105L, Q1 MMBT2222A 1P, U10 SN74AHCT125DR, U11 SN74LVC1G07DBVR, U12 MAX40200AUK+T, U2 ESP32-POE-ISO, U3 TMR 1-0511, U4 THVD1500DR, U7 6N137S, U9 SN74AHCT125DR

Commit message: Complete PCB routing with protected power bus and verified isolation
Parts:
- C8, C9: value 1uF -> 100nF
- moved R22 28.8 mm to (91.0, 63.5), turned to 180 degrees
- moved R19 25.3 mm to (70.5, 64.8), turned to 0 degrees
- moved R20 23.6 mm to (70.5, 61.0), turned to 0 degrees
- moved R21 23.4 mm to (91.0, 59.7), turned to 180 degrees
- moved R18 22.7 mm to (59.5, 63.5), turned to 180 degrees
- moved R17 19.8 mm to (59.5, 59.7), turned to 180 degrees
- moved C7 18.6 mm to (46.0, 62.0)
- moved R7 14.1 mm to (116.0, 123.2)
- moved U4 12.3 mm to (104.5, 123.0), turned to 90 degrees
- moved D1 11.2 mm to (37.0, 65.0)
- moved R16 11.2 mm to (37.0, 61.0)
- moved C11 8.38 mm to (100.8, 121.3)
- moved C14 5.50 mm to (58.5, 44.0)
- moved C15 5.50 mm to (84.5, 44.0)
- moved C16 5.50 mm to (110.5, 44.0)
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Routing:
- net +5V: track 0.00 -> 193.4 mm, vias 0 -> 20
- net 3.3V: track 0.00 -> 163.1 mm, vias 0 -> 3
- net DMX-VCC: track 0.00 -> 92.5 mm, vias 0 -> 2
- net CMD_BTN: track 0.00 -> 84.2 mm, vias 0 -> 2
- net Net-(J5-Pad4): track 0.00 -> 66.9 mm, vias 0 -> 2
- net Net-(J7-Pad2): track 0.00 -> 66.7 mm
- net Net-(J4-Pad3): track 0.00 -> 66.4 mm, vias 0 -> 2
- net GND: track 0.00 -> 63.0 mm, vias 0 -> 28
- net CAMERA_RESET_RELAY: track 0.00 -> 62.6 mm, vias 0 -> 1
- net Net-(J5-Pad3): track 0.00 -> 53.0 mm, vias 0 -> 2
- net Net-(J3-Pad3): track 0.00 -> 52.3 mm, vias 0 -> 2
- net Net-(J7-Pad1): track 0.00 -> 48.5 mm
- net 485/TX: track 0.00 -> 46.6 mm
- net PSU_LIGHT3: track 0.00 -> 45.4 mm
- net PSU_LIGHT2: track 0.00 -> 45.4 mm
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- added copper zone on F.Cu, net +5V
- added copper zone on B.Cu, net DMX-GND
- added copper zone on F.Cu, net DMX-GND
- added copper zone on B.Cu, net GND
- added copper zone on F.Cu, net GND
Other:
- board text added: "+5V"
- board text added: "3V3"
- board text added: "5 V / 8 A TOTAL MAX"
- board text added: "A"
- board text added: "B"
- board text added: "BTN"
- board text added: "C"
- board text added: "COM"
- board text added: "D"
- board text added: "ESP32-POE-ISO"
- board text added: "GND"
- board text added: "ISOLATED DMX"
- board text added: "NC"
- board text added: "PROTOTYPE / 2 oz"
- board text added: "PhotoboothHub"
- board text added: "PhotoboothHub - routed prototype"
- board text removed: "PhotoboothHub - placement draft"

Commit message: Update PCB design and 3D assets
Other:
- board size 100 x 130 mm -> 116 x 130 mm
Changed lines of the file:
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@@
 		)
 		(embedded_fonts no)
+		(model "${KIPRJMOD}/Photobooth.3dshapes/OptiFuse_CNT-06_MICRO2.step"
+			(offset
+				(xyz 0 0 0)
+			)
+			(scale
+				(xyz 1 1 1)
+			)
+			(rotate
+				(xyz 0 0 0)
+			)
+		)
 	)
 	(footprint "MountingHole:MountingHole_3.2mm_M3"
@@
 		)
 		(embedded_fonts no)
+		(model "${KIPRJMOD}/Photobooth.3dshapes/PhoenixContact_SPT_1.5_2-V-3.5_1990850.step"
+			(offset
+				(xyz 0 0 0)
+			)
+			(scale
+				(xyz 1 1 1)
+			)
+			(rotate
+				(xyz 0 0 0)
+			)
+		)
 	)
 	(footprint "Photobooth:Olimex_ESP32-POE-ISO"
 		(layer "F.Cu")
 		(at 53.22 96.71 90)
-		(descr "Olimex ESP32-POE-ISO carrier footprint; 2x10 headers, 2.54 mm pitch, 25.40 mm row spacing. Geometry verified against official Rev N1 PCB and J+ drawing; see FOOTPRINTS.md.")
-		(tags "Olimex ESP32 POE ISO carrier 25.4mm")
+		(descr "Olimex ESP32-POE-ISO removable carrier footprint; two 1x10 single-row female THT sockets, 2.54 mm pitch, 25.40 mm row spacing. Geometry verified against official Rev N1 PCB and J+ drawing; see FOOTPRINTS.md.")
+		(tags "Olimex ESP32 POE ISO carrier 1x10 socket removable 25.4mm")
 		(property "Reference" "U2"
 			(at 28.71 9.78 0)
@@
 		)
 		(embedded_fonts no)
+		(model "${KICAD10_3DMODEL_DIR}/Connector_PinSocket_2.54mm.3dshapes/PinSocket_1x10_P2.54mm_Vertical.step"
+			(offset
+				(xyz 0 0 0)
+			)
+			(scale
+				(xyz 1 1 1)
+			)
+			(rotate
+				(xyz 0 0 0)
+			)
+		)
+		(model "${KICAD10_3DMODEL_DIR}/Connector_PinSocket_2.54mm.3dshapes/PinSocket_1x10_P2.54mm_Vertical.step"
+			(offset
+				(xyz 25.4 0 0)
+			)
+			(scale
+				(xyz 1 1 1)
+			)
+			(rotate
+				(xyz 0 0 0)
+			)
+		)
+		(model "${KIPRJMOD}/Photobooth.3dshapes/ESP32-PoE-ISO_Rev_L.step"
+			(offset
+				(xyz -1.29 -64.93 8.5)
+			)
+			(scale
+				(xyz 1 1 1)
+			)
+			(rotate
+				(xyz 0 0 0)
+			)
+		)
 	)
 	(footprint "Package_DIP:SMDIP-8_W9.53mm"
@@
 		)
 		(embedded_fonts no)
+		(model "${KIPRJMOD}/Photobooth.3dshapes/OptiFuse_CNT-06_MICRO2.step"
+			(offset
+				(xyz 0 0 0)
+			)
+			(scale
+				(xyz 1 1 1)
+			)
+			(rotate
+				(xyz 0 0 0)
+			)
+		)
 	)
 	(footprint "Resistor_SMD:R_0603_1608Metric"
@@
 		)
 		(embedded_fonts no)
+		(model "${KIPRJMOD}/Photobooth.3dshapes/OptiFuse_CNT-06_MICRO2.step"
+			(offset
+				(xyz 0 0 0)
+			)
+			(scale
+				(xyz 1 1 1)
+			)
+			(rotate
+				(xyz 0 0 0)
+			)
+		)
 	)
 	(footprint "Photobooth:LED_0805_2012Metric_A1K2"
@@
 		)
 		(embedded_fonts no)
+		(model "${KIPRJMOD}/Photobooth.3dshapes/PhoenixContact_SPT_1.5_3-V-3.5_1990863.step"
+			(offset
+				(xyz 0 0 0)
+			)
+			(scale
+				(xyz 1 1 1)
+			)
+			(rotate
+				(xyz 0 0 0)
+			)
+		)
 	)
 	(footprint "Resistor_SMD:R_0603_1608Metric"
@@
 		)
 		(embedded_fonts no)
+		(model "${KIPRJMOD}/Photobooth.3dshapes/PhoenixContact_SPT_1.5_4-V-3.5_1990876.step"
+			(offset
+				(xyz 0 0 0)
+			)
+			(scale
+				(xyz 1 1 1)
+			)
+			(rotate
+				(xyz 0 0 0)
+			)
+		)
 	)
 	(footprint "Diode_SMD:D_SOD-123"
@@
 		)
 		(embedded_fonts no)
+		(model "${KIPRJMOD}/Photobooth.3dshapes/OptiFuse_CNT-06_MICRO2.step"
+			(offset
+				(xyz 0 0 0)
+			)
+			(scale
+				(xyz 1 1 1)
+			)
+			(rotate
+				(xyz 0 0 0)
+			)
+		)
 	)
 	(footprint "Capacitor_SMD:C_0603_1608Metric"
@@
 		)
 		(embedded_fonts no)
+		(model "${KIPRJMOD}/Photobooth.3dshapes/QLRELAY_BRD-SS-105L.step"
+			(offset
+				(xyz 0 0 0)
+			)
+			(scale
+				(xyz 1 1 1)
+			)
+			(rotate
+				(xyz 0 0 0)
+			)
+		)
 	)
 	(footprint "Photobooth:PhoenixContact_SPT_1.5_2-V-3.5_1990850"
@@
 		)
 		(embedded_fonts no)
+		(model "${KIPRJMOD}/Photobooth.3dshapes/PhoenixContact_SPT_1.5_2-V-3.5_1990850.step"
+			(offset
+				(xyz 0 0 0)
+			)
+			(scale
+				(xyz 1 1 1)
+			)
+			(rotate
+				(xyz 0 0 0)
+			)
+		)
 	)
 	(footprint "Photobooth:LED_0805_2012Metric_A1K2"
@@
 		)
 		(embedded_fonts no)
+		(model "${KIPRJMOD}/Photobooth.3dshapes/PhoenixContact_SPT_1.5_2-V-3.5_1990850.step"
+			(offset
+				(xyz 0 0 0)
+			)
+			(scale
+				(xyz 1 1 1)
+			)
+			(rotate
+				(xyz 0 0 0)
+			)
+		)
 	)
 	(footprint "Package_SO:SOIC-8_3.9x4.9mm_P1.27mm"
@@
 		)
 		(embedded_fonts no)
+		(model "${KIPRJMOD}/Photobooth.3dshapes/PhoenixContact_SPT_1.5_4-V-3.5_1990876.step"
+			(offset
+				(xyz 0 0 0)
+			)
+			(scale
+				(xyz 1 1 1)
+			)
+			(rotate
+				(xyz 0 0 0)
+			)
+		)
 	)
 	(footprint "Capacitor_SMD:C_0805_2012Metric"
@@
 		)
 		(embedded_fonts no)
+		(model "${KIPRJMOD}/Photobooth.3dshapes/PhoenixContact_SPT_1.5_4-V-3.5_1990876.step"
+			(offset
+				(xyz 0 0 0)
+			)
+			(scale
+				(xyz 1 1 1)
+			)
+			(rotate
+				(xyz 0 0 0)
+			)
+		)
 	)
 	(footprint "Resistor_SMD:R_0603_1608Metric"
@@
 	)
 	(gr_arc
-		(start 20 23)
-		(mid 20.87868 20.87868)
-		(end 23 20)
+		(start 12 23)
+		(mid 12.87868 20.87868)
+		(end 15 20)
 		(stroke
 			(width 0.1)
@@
 	)
 	(gr_line
-		(start 20 147)
-		(end 20 23)
+		(start 12 147)
+		(end 12 23)
 		(stroke
 			(width 0.1)
@@
 	)
 	(gr_line
-		(start 23 20)
-		(end 117 20)
+		(start 15 20)
+		(end 125 20)
 		(stroke
 			(width 0.1)
@@
 	)
 	(gr_arc
-		(start 23 150)
-		(mid 20.87868 149.12132)
-		(end 20 147)
+		(start 15 150)
+		(mid 12.87868 149.12132)
+		(end 12 147)
 		(stroke
 			(width 0.1)
@@
 	)
 	(gr_arc
-		(start 117 20)
-		(mid 119.12132 20.87868)
-		(end 120 23)
+		(start 125 20)
+		(mid 127.12132 20.87868)
+		(end 128 23)
 		(stroke
 			(width 0.1)
@@
 	)
 	(gr_line
-		(start 117 150)
-		(end 23 150)
+		(start 125 150)
+		(end 15 150)
 		(stroke
 			(width 0.1)
@@
 	)
 	(gr_line
-		(start 120 23)
-		(end 120 147)
+		(start 128 23)
+		(end 128 147)
 		(stroke
 			(width 0.1)
@@
 	)
 	(gr_arc
-		(start 120 147)
-		(mid 119.12132 149.12132)
-		(end 117 150)
+		(start 128 147)
+		(mid 127.12132 149.12132)
+		(end 125 150)
 		(stroke
 			(width 0.1)
@@
 		(polygon
 			(pts
-				(xy 20 59.46) (xy 35 59.46) (xy 35 108.56) (xy 20 108.56)
+				(xy 12 59.46) (xy 35 59.46) (xy 35 108.56) (xy 12 108.56)
 			)
 		)

Commit message: Update photobooth PCB and validation assets
Parts:
- moved C19 20.0 mm to (54.0, 84.0)
- moved C20 20.0 mm to (62.0, 84.0)
- moved U12 20.0 mm to (58.0, 84.0)
- moved R26 15.0 mm to (79.5, 117.8)
- moved C10 15.0 mm to (92.0, 121.2)
- moved C11 15.0 mm to (100.8, 106.3)
- moved C12 15.0 mm to (89.4, 105.2)
- moved C13 15.0 mm to (80.0, 105.5)
- moved C17 15.0 mm to (72.5, 117.0)
- moved C18 15.0 mm to (96.2, 108.0)
- moved D2 15.0 mm to (74.5, 122.0)
- moved H3 15.0 mm to (24.0, 131.0)
- moved H4 15.0 mm to (116.0, 131.0)
- moved J2 15.0 mm to (30.5, 122.0)
- moved J6 15.0 mm to (106.0, 115.0)
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Routing:
- net +5V: track 193.4 -> 230.1 mm
- net Net-(JP1-A): track 25.0 -> 58.1 mm
- net 3.3V: track 163.1 -> 136.4 mm
- net CAMERA_RESET_RELAY: track 62.6 -> 44.5 mm, vias 1 -> 3
- net CMD_BTN: track 84.2 -> 69.2 mm
- net 485/TX: track 46.6 -> 31.6 mm
- net Net-(D2-A): track 28.5 -> 25.5 mm
Other:
- board size 116 x 130 mm -> 116.1 x 113.5 mm
- board text removed: "5 V / 8 A TOTAL MAX"
- board text removed: "PROTOTYPE / 2 oz"
- board text removed: "PhotoboothHub"
- board text removed: "REMOVE JP1 FOR USB"
- board text removed: "USB cable access"

Commit message: Update photobooth schematic and PCB layout
Parts:
- removed R9: 120Ω, Resistor_SMD:R_0603_1608Metric
Routing:
- net DMX-VCC: track 92.5 -> 88.3 mm
- net +5V: track 230.1 -> 227.7 mm
- net GND: track 63.0 -> 60.8 mm
- net 3.3V: track 136.4 -> 134.6 mm
- net /P2/DMX-B: track 29.0 -> 27.8 mm
